File: astable-timer.kicad_sch (KiCad schematic)
At the start: 7 parts, among them U1 NE555P

Commit message: finished
Parts:
- renumbered U1 to U2
Changed lines of the file:
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@@
 		(dnp no)
 		(fields_autoplaced yes)
-		(property "Reference" "#PWR012"
+		(property "Reference" "#PWR06"
 			(at 144.78 86.36 0)
 			(effects
@@
 			(project "binary-counter"
 				(path "/9e6266cd-e24f-42f0-b90b-fa538571aa1c/d0a30e76-12cc-45f8-aea3-739e867bcd29"
-					(reference "#PWR012")
+					(reference "#PWR06")
 					(unit 1)
 				)
@@
 		(dnp no)
 		(fields_autoplaced yes)
-		(property "Reference" "U1"
+		(property "Reference" "U2"
 			(at 146.9233 86.36 0)
 			(effects
@@
 			(project "binary-counter"
 				(path "/9e6266cd-e24f-42f0-b90b-fa538571aa1c/d0a30e76-12cc-45f8-aea3-739e867bcd29"
-					(reference "U1")
+					(reference "U2")
 					(unit 1)
 				)
@@
 		(dnp no)
 		(fields_autoplaced yes)
-		(property "Reference" "#PWR013"
+		(property "Reference" "#PWR07"
 			(at 144.78 121.92 0)
 			(effects
@@
 			(project "binary-counter"
 				(path "/9e6266cd-e24f-42f0-b90b-fa538571aa1c/d0a30e76-12cc-45f8-aea3-739e867bcd29"
-					(reference "#PWR013")
-					(unit 1)
-				)
+					(reference "#PWR07")
+					(unit 1)
+				)
