File: display.kicad_sch (KiCad schematic)
At the start: 5 parts, among them U17 SM410561K, U18 74HC86, U19 SM410561K, U20 74LS248, U21 74LS83

Commit message: finished
Parts:
- removed U17, U19: SM410561K, Display_7Segment:7SegmentLED_LTS6760_LTS6780, symbol Display_Character:SM420561N
- removed U20: 74LS248, Package_DIP:DIP-16_W7.62mm_Socket, symbol 74xx:74LS248
- added AFF1, AFF2: LTS-6960HR, Display_7Segment:7SegmentLED_LTS6760_LTS6780, symbol Display_Character:LTS-6960HR
- added D4, D5, D6, D7: Red, LED_THT:LED_D5.0mm, symbol Device:LED
- added R10, R11, R12, R13, R14, R15, R16, R17, R18, R19, R20, R21: 220 R, Resistor_THT:R_Axial_DIN0207_L6.3mm_D2.5mm_P10.16mm_Horizontal, symbol Device:R_Small
- added U7: 74LS47, Package_DIP:DIP-16_W7.62mm_Socket, symbol 74xx:74LS47
- renumbered U18 to U6, U21 to U8
Connections:
- net +5V: now also AFF1.3 (C.A.), AFF1.8 (C.A.), AFF2.3 (C.A.), AFF2.8 (C.A.), U7.16 (VCC)
- net GND: now also D4.1 (K), D5.1 (K), D6.1 (K), D7.1 (K), U7.3 (LT), U7.4 (BI), U7.5 (RBI), U7.8 (GND)
- net Q0: now also R21.2
- net Q1: now also R20.2
- net Q2: now also R19.2
- net Q3: now also R18.2
- net at U6.1, U6.11, U6.4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: now also R10.1
- net at U8.15 (S4): now also U7.6 (D)
- net at U8.2 (S3): now also U7.2 (C)
- net at U8.6 (S2): now also U7.1 (B)
- net at U8.9 (S1): now also U7.7 (A)
- new net: D6.2 (A), R20.1
- new net: AFF1.10 (g), R10.2
- new net: R17.1, U7.14 (g)
- new net: AFF2.10 (g), R17.2
- new net: R14.1, U7.10 (d)
- new net: R13.1, U7.11 (c)
- new net: R12.1, U7.12 (b)
- new net: R11.1, U7.13 (a)
- new net: R16.1, U7.15 (f)
- new net: R15.1, U7.9 (e)
- new net: AFF2.1 (e), R15.2
- new net: AFF2.2 (d), R14.2
- new net: AFF2.4 (c), R13.2
- new net: AFF2.6 (b), R12.2
- new net: AFF2.7 (a), R11.2
- new net: AFF2.9 (f), R16.2
- new net: D4.2 (A), R18.1
- new net: D7.2 (A), R21.1
- new net: D5.2 (A), R19.1
- no-connect marks 2 -> 9
Other:
- moved on the sheet: U6A, U6B, U6C, U6D, U6E, U8
