File: monostable-timer.kicad_sch (KiCad schematic)
At the start: 6 parts, among them SW1 Clock, U2 NE555P

Commit message: finished
Parts:
- renumbered U2 to U3
Changed lines of the file:
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@@
 		(dnp no)
 		(fields_autoplaced yes)
-		(property "Reference" "U2"
+		(property "Reference" "U3"
 			(at 150.7333 92.71 0)
 			(effects
@@
 			(project ""
 				(path "/9e6266cd-e24f-42f0-b90b-fa538571aa1c/099caec3-6830-40cd-ab69-e1d59d4b66fc"
-					(reference "U2")
+					(reference "U3")
 					(unit 1)
 				)
@@
 		(dnp no)
 		(fields_autoplaced yes)
-		(property "Reference" "#PWR015"
+		(property "Reference" "#PWR09"
 			(at 148.59 125.73 0)
 			(effects
@@
 			(project ""
 				(path "/9e6266cd-e24f-42f0-b90b-fa538571aa1c/099caec3-6830-40cd-ab69-e1d59d4b66fc"
-					(reference "#PWR015")
+					(reference "#PWR09")
 					(unit 1)
 				)
@@
 		(dnp no)
 		(fields_autoplaced yes)
-		(property "Reference" "#PWR014"
+		(property "Reference" "#PWR08"
 			(at 148.59 92.71 0)
 			(effects
@@
 			(project ""
 				(path "/9e6266cd-e24f-42f0-b90b-fa538571aa1c/099caec3-6830-40cd-ab69-e1d59d4b66fc"
-					(reference "#PWR014")
-					(unit 1)
-				)
+					(reference "#PWR08")
+					(unit 1)
+				)
