File: timer-select.kicad_sch (KiCad schematic)
At the start: 10 parts, among them SW2 SW_SPDT, U3 74HC00, U4 NE555P

Commit message: finished
Parts:
- SW2: footprint Connector_PinHeader_1.27mm:PinHeader_1x03_P1.27mm_Vertical -> Connector_PinHeader_2.00mm:PinHeader_1x03_P2.00mm_Vertical
- renumbered U3 to U4, U4 to U5
Changed lines of the file:
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@@
 		(dnp no)
 		(fields_autoplaced yes)
-		(property "Reference" "U3"
+		(property "Reference" "U4"
 			(at 238.76 96.5199 0)
 			(effects
@@
 			(project ""
 				(path "/9e6266cd-e24f-42f0-b90b-fa538571aa1c/f09e22f1-de7b-49af-bc53-06aaa0ad2632"
-					(reference "U3")
+					(reference "U4")
 					(unit 5)
 				)
@@
 		(dnp no)
 		(fields_autoplaced yes)
-		(property "Reference" "U4"
+		(property "Reference" "U5"
 			(at 113.9033 87.63 0)
 			(effects
@@
 			(project "binary-counter"
 				(path "/9e6266cd-e24f-42f0-b90b-fa538571aa1c/f09e22f1-de7b-49af-bc53-06aaa0ad2632"
-					(reference "U4")
+					(reference "U5")
 					(unit 1)
 				)
@@
 		(dnp no)
 		(fields_autoplaced yes)
-		(property "Reference" "U3"
+		(property "Reference" "U4"
 			(at 194.3017 90.17 0)
 			(effects
@@
 			(project ""
 				(path "/9e6266cd-e24f-42f0-b90b-fa538571aa1c/f09e22f1-de7b-49af-bc53-06aaa0ad2632"
-					(reference "U3")
+					(reference "U4")
 					(unit 4)
 				)
@@
 		(dnp no)
 		(fields_autoplaced yes)
-		(property "Reference" "#PWR017"
+		(property "Reference" "#PWR011"
 			(at 232.41 87.63 0)
 			(effects
@@
 			(project "binary-counter"
 				(path "/9e6266cd-e24f-42f0-b90b-fa538571aa1c/f09e22f1-de7b-49af-bc53-06aaa0ad2632"
-					(reference "#PWR017")
+					(reference "#PWR011")
 					(unit 1)
 				)
@@
 		(dnp no)
 		(fields_autoplaced yes)
-		(property "Reference" "U3"
+		(property "Reference" "U4"
 			(at 154.9317 83.82 0)
 			(effects
@@
 			(project ""
 				(path "/9e6266cd-e24f-42f0-b90b-fa538571aa1c/f09e22f1-de7b-49af-bc53-06aaa0ad2632"
-					(reference "U3")
+					(reference "U4")
 					(unit 1)
 				)
@@
 		(dnp no)
 		(fields_autoplaced yes)
-		(property "Reference" "#PWR018"
+		(property "Reference" "#PWR012"
 			(at 232.41 118.11 0)
 			(effects
@@
 			(project "binary-counter"
 				(path "/9e6266cd-e24f-42f0-b90b-fa538571aa1c/f09e22f1-de7b-49af-bc53-06aaa0ad2632"
-					(reference "#PWR018")
+					(reference "#PWR012")
 					(unit 1)
 				)
@@
 		(dnp no)
 		(fields_autoplaced yes)
-		(property "Reference" "#PWR016"
+		(property "Reference" "#PWR010"
 			(at 111.76 86.36 0)
 			(effects
@@
 			(project ""
 				(path "/9e6266cd-e24f-42f0-b90b-fa538571aa1c/f09e22f1-de7b-49af-bc53-06aaa0ad2632"
-					(reference "#PWR016")
+					(reference "#PWR010")
 					(unit 1)
 				)
@@
 		(dnp no)
 		(fields_autoplaced yes)
-		(property "Reference" "#PWR019"
+		(property "Reference" "#PWR013"
 			(at 111.76 120.65 0)
 			(effects
@@
 			(project ""
 				(path "/9e6266cd-e24f-42f0-b90b-fa538571aa1c/f09e22f1-de7b-49af-bc53-06aaa0ad2632"
-					(reference "#PWR019")
+					(reference "#PWR013")
 					(unit 1)
 				)
@@
 		(dnp no)
 		(fields_autoplaced yes)
-		(property "Reference" "U3"
+		(property "Reference" "U4"
 			(at 154.9317 99.06 0)
 			(effects
@@
 			(project ""
 				(path "/9e6266cd-e24f-42f0-b90b-fa538571aa1c/f09e22f1-de7b-49af-bc53-06aaa0ad2632"
-					(reference "U3")
+					(reference "U4")
 					(unit 2)
 				)
@@
 		(dnp no)
 		(fields_autoplaced yes)
-		(property "Reference" "U3"
+		(property "Reference" "U4"
 			(at 176.5217 96.52 0)
 			(effects
@@
 			(project ""
 				(path "/9e6266cd-e24f-42f0-b90b-fa538571aa1c/f09e22f1-de7b-49af-bc53-06aaa0ad2632"
-					(reference "U3")
+					(reference "U4")
 					(unit 3)
 				)
@@
 			)
 		)
-		(property "Footprint" "Connector_PinHeader_1.27mm:PinHeader_1x03_P1.27mm_Vertical"
+		(property "Footprint" "Connector_PinHeader_2.00mm:PinHeader_1x03_P2.00mm_Vertical"
 			(at 78.74 100.33 0)
 			(effects

Commit message: the end
Parts:
- SW2: footprint Connector_PinHeader_2.00mm:PinHeader_1x03_P2.00mm_Vertical -> Switches:IC-205
Changed lines of the file:
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@@
 			)
 		)
-		(property "Footprint" "Connector_PinHeader_2.00mm:PinHeader_1x03_P2.00mm_Vertical"
+		(property "Footprint" "Switches:IC-205"
 			(at 78.74 100.33 0)
 			(effects
